Commit message: change STL to stl

File: simulation/assets/humanoid_urdf/humanoid.urdf (robot description, URDF)
Before this commit: robot new_humanoid1, 13 links, 12 joints
Links:
- link left_forearm_pitch_link: geometry collision mesh filename=package://new_humanoid1/meshes/left_forearm_pitch_link.stl; visual mesh filename=package://new_humanoid1/meshes/left_forearm_pitch_link.stl
- link left_knee_pitch_link: geometry collision mesh filename=package://new_humanoid1/meshes/left_knee_pitch_link.stl; visual mesh filename=package://new_humanoid1/meshes/left_knee_pitch_link.stl
- link left_shoulder_pitch_link: geometry collision mesh filename=package://new_humanoid1/meshes/left_shoulder_pitch_link.stl; visual mesh filename=package://new_humanoid1/meshes/left_shoulder_pitch_link.stl
- link left_shoulder_roll_link: geometry collision mesh filename=package://new_humanoid1/meshes/left_shoulder_roll_link.stl; visual mesh filename=package://new_humanoid1/meshes/left_shoulder_roll_link.stl
- link left_waist_pitch_link: geometry collision mesh filename=package://new_humanoid1/meshes/left_waist_pitch_link.stl; visual mesh filename=package://new_humanoid1/meshes/left_waist_pitch_link.stl
- link left_waist_roll_link: geometry collision mesh filename=package://new_humanoid1/meshes/left_waist_roll_link.stl; visual mesh filename=package://new_humanoid1/meshes/left_waist_roll_link.stl
- link right_forearm_pitch_link: geometry collision mesh filename=package://new_humanoid1/meshes/right_forearm_pitch_link.stl; visual mesh filename=package://new_humanoid1/meshes/right_forearm_pitch_link.stl
- link right_knee_pitch_link: geometry collision mesh filename=package://new_humanoid1/meshes/right_knee_pitch_link.stl; visual mesh filename=package://new_humanoid1/meshes/right_knee_pitch_link.stl
- link right_shoulder_pitch_link: geometry collision mesh filename=package://new_humanoid1/meshes/right_shoulder_pitch_link.stl; visual mesh filename=package://new_humanoid1/meshes/right_shoulder_pitch_link.stl
- link right_shoulder_roll_link: geometry collision mesh filename=package://new_humanoid1/meshes/right_shoulder_roll_link.stl; visual mesh filename=package://new_humanoid1/meshes/right_shoulder_roll_link.stl
- link right_waist_pitch_link: geometry collision mesh filename=package://new_humanoid1/meshes/right_waist_pitch_link.stl; visual mesh filename=package://new_humanoid1/meshes/right_waist_pitch_link.stl
- link right_waist_roll_link: geometry collision mesh filename=package://new_humanoid1/meshes/right_waist_roll_link.stl; visual mesh filename=package://new_humanoid1/meshes/right_waist_roll_link.stl
- link torso: geometry collision mesh filename=package://new_humanoid1/meshes/torso.stl; visual mesh filename=package://new_humanoid1/meshes/torso.stl

Commit message: convert mujoco xmls to urdfs

File: simulation/assets/humanoid_urdf/humanoid.urdf (robot description, URDF)
Before this commit: robot new_humanoid1, 13 links, 12 joints
Joints:
- joint left_forearm_pitch_joint: type continuous -> revolute
- joint left_knee_pitch_joint: type continuous -> revolute
- joint left_shoulder_pitch_joint: type continuous -> revolute
- joint left_shoulder_roll_joint: type continuous -> revolute
- joint left_waist_pitch_joint: type continuous -> revolute
- joint left_waist_roll_joint: type continuous -> revolute
- joint right_forearm_pitch_joint: type continuous -> revolute
- joint right_knee_pitch_joint: type continuous -> revolute
- joint right_shoulder_pitch_joint: type continuous -> revolute
- joint right_shoulder_roll_joint: type continuous -> revolute
- joint right_waist_pitch_joint: type continuous -> revolute
- joint right_waist_roll_joint: type continuous -> revolute
