Commit message: add floor and collisions to world

File: id_urdf/world.urdf (robot description, URDF)
Before this commit: robot new_humanoid1, 31 links, 30 joints
Links:
- added link floor; collision box size=100 100 0.01; visual box size=100 100 0.1
- link left_forearm_pitch_link: geometry collision mesh filename=/root/Humanoid-MuJoCo-Inverse-Dynamics/id_urdf/converted_le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; visual mesh filename=/root/Humanoid-MuJoCo-Inverse-Dynamics/id_urdf/converted_le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
- link left_knee_pitch_link: geometry collision mesh filename=/root/Humanoid-MuJoCo-Inverse-Dynamics/id_urdf/converted_ri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; visual mesh filename=/root/Humanoid-MuJoCo-Inverse-Dynamics/id_urdf/converted_ri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
- link left_shoulder_pitch_link: geometry collision mesh filename=/root/Humanoid-MuJoCo-Inverse-Dynamics/id_urdf/converted_le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; visual mesh filename=/root/Humanoid-MuJoCo-Inverse-Dynamics/id_urdf/converted_le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
- link left_waist_pitch_link: geometry collision mesh filename=/root/Humanoid-MuJoCo-Inverse-Dynamics/id_urdf/converted_ri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; visual mesh filename=/root/Humanoid-MuJoCo-Inverse-Dynamics/id_urdf/converted_ri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
- link right_forearm_pitch_link: geometry collision mesh filename=/root/Humanoid-MuJoCo-Inverse-Dynamics/id_urdf/converted_le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; visual mesh filename=/root/Humanoid-MuJoCo-Inverse-Dynamics/id_urdf/converted_le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
- link right_knee_pitch_link: geometry collision mesh filename=/root/Humanoid-MuJoCo-Inverse-Dynamics/id_urdf/converted_le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; visual mesh filename=/root/Humanoid-MuJoCo-Inverse-Dynamics/id_urdf/converted_le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
- link right_shoulder_pitch_link: geometry collision mesh filename=/root/Humanoid-MuJoCo-Inverse-Dynamics/id_urdf/converted_le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; visual mesh filename=/root/Humanoid-MuJoCo-Inverse-Dynamics/id_urdf/converted_le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
- link right_waist_pitch_link: geometry collision mesh filename=/root/Humanoid-MuJoCo-Inverse-Dynamics/id_urdf/converted_le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; visual mesh filename=/root/Humanoid-MuJoCo-Inverse-Dynamics/id_urdf/converted_le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
- link torso: geometry collision mesh filename=/root/Humanoid-MuJoCo-Inverse-Dynamics/id_urdf/converted_to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; visual mesh filename=/root/Humanoid-MuJoCo-Inverse-Dynamics/id_urdf/converted_to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
Joints:
- added joint fixed_floor: type fixed, parent world, child floor, origin xyz=0 0 0 rpy=0 0 0

Commit message: make floor in correct position world.urdf

File: id_urdf/world.urdf (robot description, URDF)
Before this commit: robot new_humanoid1, 32 links, 31 joints
Joints:
- joint fixed_floor: origin xyz=0 0 0 rpy=0 0 0 -> xyz=0 0 -0.375 rpy=0 0 0
