Commit message: good state

File: id_urdf/humanoid.urdf (robot description, URDF)
Before this commit: robot converted_robot, 31 links, 30 joints
Links:
- link left_forearm_pitch_link: geometry visual mesh filename=/root/Humanoid-MuJoCo-Inverse-Dynamics/id_urdf/converted_le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
- link left_knee_pitch_link: geometry visual mesh filename=/root/Humanoid-MuJoCo-Inverse-Dynamics/id_urdf/converted_ri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
- link left_shoulder_pitch_link: geometry visual mesh filename=/root/Humanoid-MuJoCo-Inverse-Dynamics/id_urdf/converted_le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
- link left_waist_pitch_link: geometry visual mesh filename=/root/Humanoid-MuJoCo-Inverse-Dynamics/id_urdf/converted_ri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
- link right_forearm_pitch_link: geometry visual mesh filename=/root/Humanoid-MuJoCo-Inverse-Dynamics/id_urdf/converted_le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
- link right_knee_pitch_link: geometry visual mesh filename=/root/Humanoid-MuJoCo-Inverse-Dynamics/id_urdf/converted_le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
- link right_shoulder_pitch_link: geometry visual mesh filename=/root/Humanoid-MuJoCo-Inverse-Dynamics/id_urdf/converted_le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
- link right_waist_pitch_link: geometry visual mesh filename=/root/Humanoid-MuJoCo-Inverse-Dynamics/id_urdf/converted_le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
- link torso: geometry visual mesh filename=/root/Humanoid-MuJoCo-Inverse-Dynamics/id_urdf/converted_to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

File: simulation/assets/humanoid_urdf/humanoid.urdf (robot description, URDF)
Before this commit: robot new_humanoid1, 13 links, 12 joints
Links:
- link left_forearm_pitch_link: geometry collision mesh filename=/root/Humanoid-MuJoCo-Inverse-Dynamics/simulation/assets/hu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; visual mesh filename=/root/Humanoid-MuJoCo-Inverse-Dynamics/simulation/assets/hu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
- link left_knee_pitch_link: geometry collision mesh filename=/root/Humanoid-MuJoCo-Inverse-Dynamics/simulation/assets/hu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; visual mesh filename=/root/Humanoid-MuJoCo-Inverse-Dynamics/simulation/assets/hu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
- link left_shoulder_pitch_link: geometry collision mesh filename=/root/Humanoid-MuJoCo-Inverse-Dynamics/simulation/assets/hu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; visual mesh filename=/root/Humanoid-MuJoCo-Inverse-Dynamics/simulation/assets/hu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
- link left_shoulder_roll_link: geometry collision mesh filename=/root/Humanoid-MuJoCo-Inverse-Dynamics/simulation/assets/hu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; visual mesh filename=/root/Humanoid-MuJoCo-Inverse-Dynamics/simulation/assets/hu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
- link left_waist_pitch_link: geometry collision mesh filename=/root/Humanoid-MuJoCo-Inverse-Dynamics/simulation/assets/hu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; visual mesh filename=/root/Humanoid-MuJoCo-Inverse-Dynamics/simulation/assets/hu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
- link left_waist_roll_link: geometry collision mesh filename=/root/Humanoid-MuJoCo-Inverse-Dynamics/simulation/assets/hu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; visual mesh filename=/root/Humanoid-MuJoCo-Inverse-Dynamics/simulation/assets/hu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
- link right_forearm_pitch_link: geometry collision mesh filename=/root/Humanoid-MuJoCo-Inverse-Dynamics/simulation/assets/hu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; visual mesh filename=/root/Humanoid-MuJoCo-Inverse-Dynamics/simulation/assets/hu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
- link right_knee_pitch_link: geometry collision mesh filename=/root/Humanoid-MuJoCo-Inverse-Dynamics/simulation/assets/hu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; visual mesh filename=/root/Humanoid-MuJoCo-Inverse-Dynamics/simulation/assets/hu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
- link right_shoulder_pitch_link: geometry collision mesh filename=/root/Humanoid-MuJoCo-Inverse-Dynamics/simulation/assets/hu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; visual mesh filename=/root/Humanoid-MuJoCo-Inverse-Dynamics/simulation/assets/hu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
- link right_shoulder_roll_link: geometry collision mesh filename=/root/Humanoid-MuJoCo-Inverse-Dynamics/simulation/assets/hu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; visual mesh filename=/root/Humanoid-MuJoCo-Inverse-Dynamics/simulation/assets/hu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
- link right_waist_pitch_link: geometry collision mesh filename=/root/Humanoid-MuJoCo-Inverse-Dynamics/simulation/assets/hu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; visual mesh filename=/root/Humanoid-MuJoCo-Inverse-Dynamics/simulation/assets/hu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
- link right_waist_roll_link: geometry collision mesh filename=/root/Humanoid-MuJoCo-Inverse-Dynamics/simulation/assets/hu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; visual mesh filename=/root/Humanoid-MuJoCo-Inverse-Dynamics/simulation/assets/hu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
- link torso: geometry collision mesh filename=/root/Humanoid-MuJoCo-Inverse-Dynamics/simulation/assets/hu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; visual mesh filename=/root/Humanoid-MuJoCo-Inverse-Dynamics/simulation/assets/hu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
Joints:
- joint left_forearm_pitch_joint: type revolute -> continuous
- joint left_knee_pitch_joint: type revolute -> continuous
- joint left_shoulder_pitch_joint: type revolute -> continuous
- joint left_shoulder_roll_joint: type revolute -> continuous
- joint left_waist_pitch_joint: type revolute -> continuous
- joint left_waist_roll_joint: type revolute -> continuous
- joint right_forearm_pitch_joint: type revolute -> continuous
- joint right_knee_pitch_joint: type revolute -> continuous
- joint right_shoulder_pitch_joint: type revolute -> continuous
- joint right_shoulder_roll_joint: type revolute -> continuous
- joint right_waist_pitch_joint: type revolute -> continuous
- joint right_waist_roll_joint: type revolute -> continuous

Commit message: its moving, but not well

File: id_urdf/humanoid.urdf (robot description, URDF)
Before this commit: robot new_humanoid1, 31 links, 30 joints
Links:
- removed link world2humanoid_world_link_fixed_jointbody
- added link floating_base, mass 1
- link world: mass 0.0 -> None
Joints:
- removed joint world2humanoid_world_link_fixed
- removed joint world2humanoid_world_link_fixed_offset
- added joint floating_base_to_humanoid: type fixed, parent floating_base, child humanoid_world_link, origin xyz=0 0 0 rpy=0 0 0
- added joint floating_joint: type floating, parent world, child floating_base

Commit message: got skeleton code in a really good spot for optimal control

File: id_urdf/humanoid.urdf (robot description, URDF)
Before this commit: robot new_humanoid1, 31 links, 30 joints
Links:
- added link floor; collision box size=100 100 0.01; visual box size=100 100 0.01
- link left_forearm_pitch_link: geometry collision mesh filename=/root/Humanoid-MuJoCo-Inverse-Dynamics/id_urdf/converted_le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; visual mesh filename=/root/Humanoid-MuJoCo-Inverse-Dynamics/id_urdf/converted_le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
- link left_knee_pitch_link: geometry collision mesh filename=/root/Humanoid-MuJoCo-Inverse-Dynamics/id_urdf/converted_ri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; visual mesh filename=/root/Humanoid-MuJoCo-Inverse-Dynamics/id_urdf/converted_ri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
- link left_shoulder_pitch_link: geometry collision mesh filename=/root/Humanoid-MuJoCo-Inverse-Dynamics/id_urdf/converted_le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; visual mesh filename=/root/Humanoid-MuJoCo-Inverse-Dynamics/id_urdf/converted_le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
- link left_waist_pitch_link: geometry collision mesh filename=/root/Humanoid-MuJoCo-Inverse-Dynamics/id_urdf/converted_ri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; visual mesh filename=/root/Humanoid-MuJoCo-Inverse-Dynamics/id_urdf/converted_ri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
- link right_forearm_pitch_link: geometry collision mesh filename=/root/Humanoid-MuJoCo-Inverse-Dynamics/id_urdf/converted_le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; visual mesh filename=/root/Humanoid-MuJoCo-Inverse-Dynamics/id_urdf/converted_le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
- link right_knee_pitch_link: geometry collision mesh filename=/root/Humanoid-MuJoCo-Inverse-Dynamics/id_urdf/converted_le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; visual mesh filename=/root/Humanoid-MuJoCo-Inverse-Dynamics/id_urdf/converted_le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
- link right_shoulder_pitch_link: geometry collision mesh filename=/root/Humanoid-MuJoCo-Inverse-Dynamics/id_urdf/converted_le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; visual mesh filename=/root/Humanoid-MuJoCo-Inverse-Dynamics/id_urdf/converted_le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
- link right_waist_pitch_link: geometry collision mesh filename=/root/Humanoid-MuJoCo-Inverse-Dynamics/id_urdf/converted_le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; visual mesh filename=/root/Humanoid-MuJoCo-Inverse-Dynamics/id_urdf/converted_le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
- link torso: geometry collision mesh filename=/root/Humanoid-MuJoCo-Inverse-Dynamics/id_urdf/converted_to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; visual mesh filename=/root/Humanoid-MuJoCo-Inverse-Dynamics/id_urdf/converted_to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
Joints:
- added joint fixed_floor: type fixed, parent world, child floor, origin xyz=0 0 -0.375 rpy=0 0 0
